File: two_layer_node_board/two_layer_node_board.kicad_sch (KiCad schematic)
At the start: 59 parts, among them J1 Screw_Terminal_01x04, J10 Conn_01x03_Pin, J11 Conn_01x03_Socket, J12 Conn_01x03_Socket, J2 Conn_01x03_Pin, J3 Conn_01x03_Pin, J4 Screw_Terminal_01x04, J5 Screw_Terminal_01x03, J6 Screw_Terminal_01x03, J7 Screw_Terminal_01x03, J8 Screw_Terminal_01x03, J9 Conn_01x03_Pin, SW1 SW_MEC_5E, SW2 SW_MEC_5E, U1 THVD1450D, U2 LM7805_TO220, U3 ME6211C33M5, U4 RP2040, U5 W25Q32JVSS, Y1 Crystal

Commit message: AI question for next phase of the project
Parts:
- removed R10: 120, symbol Device:R
- added JP1: Jumper_2_Open, symbol Jumper:Jumper_2_Open
- added R11: 120, symbol Device:R
Connections:
- net +12V: now also D2.2 (A); no longer D2.1 (K)
- net GND: now also D2.1 (K); no longer D2.2 (A)
- net RS485_A: now also R11.2
- net RS485_B: now also U1.7 (B), JP1.2 (B)
- net +3V3_MCU: now reaches U4.1 (IOVDD), U4.10 (IOVDD), U4.22 (IOVDD), U4.33 (IOVDD), U4.42 (IOVDD), U4.43 (ADC_AVDD), U4.48 (USB_VDD), U4.49 (IOVDD)
- new net: JP1.1 (A), R11.1
Other:
- moved on the sheet: D2

Commit message: arduino-nano-node-version
Parts:
- removed C11: 10pF, symbol Device:C
- removed C12: .1uF, symbol Device:C
- removed C13, C18: 1uF, symbol Device:C
- removed C14, C15, C16, C17, C19, C20, C21: 0.1uF, symbol Device:C
- removed C22, C23, C24, C25, C8: 220uF, symbol Device:C
- removed C3: 10uF, symbol Device:C
- removed C4: 22uF, symbol Device:C
- removed J11, J12: Conn_01x03_Socket, symbol Connector:Conn_01x03_Socket
- removed J2: Conn_01x03_Pin, Connector_PinHeader_2.54mm:PinHeader_1x03_P2.54mm_Vertical, symbol Connector:Conn_01x03_Pin
- removed J4: Screw_Terminal_01x04, symbol Connector:Screw_Terminal_01x04
- removed J5, J6, J7, J8: Screw_Terminal_01x03, symbol Connector:Screw_Terminal_01x03
- removed JP1: Jumper_2_Open, symbol Jumper:Jumper_2_Open
- removed R3, R4, R5, R6, R9: 10k, symbol Device:R
- removed R7: 1M, symbol Device:R
- removed R8: 220, symbol Device:R
- removed SW1, SW2: SW_MEC_5E, symbol Switch:SW_MEC_5E
- removed U2: LM7805_TO220, Package_TO_SOT_THT:TO-220-3_Vertical, symbol Regulator_Linear:LM7805_TO220
- removed U4: RP2040, Package_DFN_QFN:QFN-56-1EP_7x7mm_P0.4mm_EP3.2x3.2mm, symbol MCU_RaspberryPi:RP2040
- removed U5: W25Q32JVSS, Package_SO:SOIC-8_5.3x5.3mm_P1.27mm, symbol Memory_Flash:W25Q32JVSS
- removed Y1: Crystal, symbol Device:Crystal
- added A1: Arduino_Nano_Every, Module:Arduino_Nano, symbol MCU_Module:Arduino_Nano_Every
- added C8: C_Polarized, symbol Device:C_Polarized
- added J13, J18, J19, J20, J21: Conn_01x03_Pin, symbol Connector:Conn_01x03_Pin
- added J2: Screw_Terminal_01x02, symbol Connector:Screw_Terminal_01x02
- added J27, J28, J29, J4: Conn_01x04_Pin, symbol Connector:Conn_01x04_Pin
- added JP1, JP10, JP11, JP12, JP13, JP2, JP4, JP5, JP6, JP7, JP8, JP9: SolderJumper_2_Open, symbol Jumper:SolderJumper_2_Open
- added Q2: IRLML6401, Package_TO_SOT_SMD:SOT-23, symbol Transistor_FET:IRLML6401
- added R10, R15, R17, R18, R23, R24, R25, R35, R36, R39, R41, R43, R44, R45, R47: 10k, symbol Device:R
- added R12, R13, R14, R16, R27, R28, R29, R30: 220, symbol Device:R
- added R37, R38: 4.7k, symbol Device:R
- added R48, R7, R8 (x2): 10K, Adafruit PCA9685:0805, symbol Adafruit PCA9685-eagle-import:RESISTOR0805
- added U4, U7: PCA9685PW, Package_SO:TSSOP-28_4.4x9.7mm_P0.65mm, symbol Driver_LED:PCA9685PW
- added U6, U8: CD74HC4067M, Package_SO:SOIC-24W_7.5x15.4mm_P1.27mm, symbol 74xx:CD74HC4067M
- C10: value 10pF -> 10uF
- C9: value 220uF -> 10uF
- J10, J3, J9: footprint Connector_PinHeader_2.54mm:PinHeader_1x03_P2.54mm_Vertical -> (none)
Connections:
- net +5V: now also C1.1, C2.1, U1.8 (VCC), R37.1; no longer C5.1, C9.2, J10.2 (Pin_2), J3.2 (Pin_2), J9.2 (Pin_2), U3.1 (V_{IN}), U3.3 (CE)
- net GND: now also C9.2, A1.29 (GND), A1.4 (GND), C8.2, J13.1 (Pin_1), J18.1 (Pin_1), J19.1 (Pin_1), J2.2 (Pin_2), J20.1 (Pin_1), J21.1 (Pin_1), J27.4 (Pin_4), J28.4 (Pin_4), J29.4 (Pin_4), J4.4 (Pin_4), Q2.1 (G), R15.2, R17.2, R18.2, R23.2, R24.2, R25.2, R38.2, R39.2, R41.2, R43.2, R44.2, R45.2, R47.2, U4.14 (VSS), U6.12 (GND), U7.14 (VSS), U8.12 (GND); no longer C10.1, C9.1
- net RS485_A: now also R37.2
- net RS485_B: now also JP1.1 (A), R38.1
- net RS485_RE_DE: now also A1.5 (D2)
- net at R11.1: now also JP1.2 (B)
- net +3.3V: no longer names the net of C6.1, C7.1, R1.1, U3.5 (V_{OUT})
- net +3.3V: no longer C1.1, C2.1, R2.1, U1.8 (VCC)
- net Buck In renamed +12V_BUCK_PROT
- net +12V_BUCK_PROT: now also J27.3 (Pin_3), J28.3 (Pin_3), J29.3 (Pin_3), J4.3 (Pin_3)
- net FAN_TACH renamed FAN0_VFG
- net FAN0_VFG: now also J4.2 (Pin_2)
- net SERVO_WINDOW_X_OPPO_PWM: no longer names the net of J9.3 (Pin_3)
- net SERVO_WINDOW_X_OPPO_PWM: now also R12.2
- net SERVO_WINDOW_Y_OPPO_PWM: no longer names the net of J10.3 (Pin_3)
- net SERVO_WINDOW_Y_OPPO_PWM: now also R13.2
- net SERVO_WINDOW_Y_SAME_PWM: no longer names the net of J3.3 (Pin_3)
- net SERVO_WINDOW_Y_SAME_PWM: now also R16.2
- net UART RX renamed RS485_RX
- net RS485_RX: now also A1.2 (RX1)
- net UART TX renamed RS485_TX
- net RS485_TX: now also A1.1 (TX1)
- new net: C8.1, Q2.3 (D)
- new net: J13.3 (Pin_3), R14.2
- new net: J21.3 (Pin_3), R30.2
- new net: J18.3 (Pin_3), R27.2
- new net: J2.1 (Pin_1), Q2.2 (S)
- new net: J19.3 (Pin_3), R28.2
- new net: J20.3 (Pin_3), R29.2
- new net +3V3: A1.17 (3V3)
- new net +5V_A: A1.27 (+5V), C5.1, C9.1, J10.2 (Pin_2), J13.2 (Pin_2), J18.2 (Pin_2), J19.2 (Pin_2), J20.2 (Pin_2), J21.2 (Pin_2), J9.2 (Pin_2), JP10.1 (A), JP11.1 (A), JP12.1 (A), JP13.1 (A), JP4.1 (A), R47.1, R48.2, R8.2, R8.2, U3.1 (V_{IN}), U3.3 (CE), U4.1 (A0), U4.28 (VDD), U6.24 (VCC), U8.24 (VCC)
- new net +5V_B: C10.1, J3.2 (Pin_2), R10.1, R2.1, R35.1, R36.1, R7.2, U7.28 (VDD)
- new net ANEM0: U6.9 (I0)
- new net ANEM1: U6.8 (I1)
- new net ANEM10: U6.21 (I10)
- new net ANEM11: U6.20 (I11)
- new net ANEM12: U6.19 (I12)
- new net ANEM13: U6.18 (I13)
- new net ANEM14: U6.17 (I14)
- new net ANEM15: U6.16 (I15)
- new net ANEM2: U6.7 (I2)
- new net ANEM3: U6.6 (I3)
- new net ANEM4: U6.5 (I4)
- new net ANEM5: U6.4 (I5)
- new net ANEM6: U6.3 (I6)
- new net ANEM7: U6.2 (I7)
- new net ANEM8: U6.23 (I8)
- new net ANEM9: U6.22 (I9)
- new net ANEM_PICK: U6.1 (COM)
- new net FAN0_PWM: J4.1 (Pin_1)
- new net FAN1_PWM: J27.1 (Pin_1)
- new net FAN1_VFG: J27.2 (Pin_2), R10.2
- new net FAN2_PWM: J28.1 (Pin_1)
- new net FAN2_VFG: J28.2 (Pin_2), R35.2
- new net FAN3_PWM: J29.1 (Pin_1)
- new net FAN3_VFG: J29.2 (Pin_2), R36.2
- new net FAN_A1: JP4.2 (B), JP5.2 (B), R15.1, R45.1, U4.2 (A1), U7.2 (A1)
- new net FAN_A2: JP10.2 (B), JP6.2 (B), R18.1, R44.1, U4.3 (A2), U7.3 (A2)
- new net FAN_A3: JP11.2 (B), JP7.2 (B), R23.1, R43.1, U4.4 (A3), U7.4 (A3)
- new net FAN_A4: JP12.2 (B), JP8.2 (B), R24.1, R41.1, U4.5 (A4), U7.5 (A4)
- new net FAN_A5: JP13.2 (B), JP9.2 (B), R25.1, R39.1, U4.24 (A5), U7.24 (A5)
- new net OE: R48.1, R7.1, U4.23 (~{OE}), U7.23 (~{OE})
- new net PWM0: R30.1, U4.6 (LED0), U7.6 (LED0)
- new net PWM1: R29.1, U4.7 (LED1), U7.7 (LED1)
- new net PWM10: U4.17 (LED10), U7.17 (LED10)
- new net PWM11: U4.18 (LED11), U7.18 (LED11)
- new net PWM12: U4.19 (LED12), U7.19 (LED12)
- new net PWM13: U4.20 (LED13), U7.20 (LED13)
- new net PWM14: U4.21 (LED14), U7.21 (LED14)
- new net PWM15: U4.22 (LED15), U7.22 (LED15)
- new net PWM2: R28.1, U4.8 (LED2), U7.8 (LED2)
- new net PWM3: R27.1, U4.9 (LED3), U7.9 (LED3)
- new net PWM4: R14.1, U4.10 (LED4), U7.10 (LED4)
- new net PWM5: R13.1, U4.11 (LED5), U7.11 (LED5)
- new net PWM6: R12.1, U4.12 (LED6), U7.12 (LED6)
- new net PWM7: R16.1, U4.13 (LED7), U7.13 (LED7)
- new net PWM8: U4.15 (LED8), U7.15 (LED8)
- new net PWM9: U4.16 (LED9), U7.16 (LED9)
- new net S0: A1.10 (D7), U6.10 (S0), U8.10 (S0)
- new net S1: A1.11 (D8), U6.11 (S1), U8.11 (S1)
- new net S2: A1.12 (D9), U6.14 (S2), U8.14 (S2)
- new net S3: A1.13 (D10), U6.13 (S3), U8.13 (S3)
- new net SCL: A1.24 (SCL/A5), R8.1, U4.26 (SCL), U7.26 (SCL)
- new net SDA: A1.23 (SDA/A4), R8.1, U4.27 (SDA), U7.27 (SDA)
- new net SERVO_A0: JP2.2 (B), R17.1, U7.1 (A0)
- new net TELEM_PICK: A1.19 (A0)
- new net TEMP_HUM_PICK: U8.1 (COM)
- new net TEMP/HUM0: U8.16 (I15), U8.17 (I14), U8.18 (I13), U8.19 (I12), U8.2 (I7), U8.20 (I11), U8.21 (I10), U8.22 (I9), U8.23 (I8), U8.3 (I6), U8.4 (I5), U8.9 (I0)
- new net TEMP/HUM1: U8.8 (I1)
- new net TEMP/HUM2: U8.7 (I2)
- new net TEMP/HUM3: U8.6 (I3)
- new net TEMP/HUM4: U8.5 (I4)
- new net TH_ANEM_VFG_0: A1.8 (D5)
- new net TH_ANEM_VFG_1: A1.9 (D6)
- new net VCC: JP2.1 (A), JP5.1 (A), JP6.1 (A), JP7.1 (A), JP8.1 (A), JP9.1 (A)
- no-connect marks 17 -> 26
Other:
- note added: "1 + A5 + A4 + A3 + A2 + A1 +A1 + RW"
- note added: "Add to multiplexer for temp/hum vs anemometer"
- note added: "Anemometer telemetry"
- note added: "Controls the 4-wire fans"
- note added: "Controls the Servos"
- note added: "I2C Address ="
- note added: "Open = 0 / Closed = 1"
- note added: "Reverse voltage"
- note added: "Temp and humidity telemetry"
- note added: "This I2C address is 0x40"
- note added: "This I2C address is 0x41"
- note added: "protection"
- note removed: "Boot"
- note removed: "Buck Converter"
- note removed: "Crystal"
- note removed: "DHT11_SENSOR_PORT"
- note removed: "Node outputs controls set by Master"
- note removed: "Pully Servo Connection"
- note removed: "Reset"
- note removed: "Window Servo Connection"
- moved on the sheet: C1, C2, R2
